File: circuit/mems_lora/mems_lora.kicad_sch (KiCad schematic)
At the start: 39 parts, among them J1 Conn_01x02_Pin, J2 Conn_01x05_Pin, J3 Conn_01x03_Pin, J4 Conn_01x04_Pin, SW1 SW_Push, SW2 SW_Push, U1 AMS1117-3.3, U2 TE-830M1-0025, U3 STM32F103RBTx, U4 Ai-Thinker-Ra-02

Commit message: soldering drive me crazy
Parts:
- R3: value 10K -> DNP
Changed lines of the file:
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@@
       (effects (font (size 1.27 1.27)) (justify left))
     )
-    (property "Value" "10K" (at 214.63 93.98 90)
+    (property "Value" "DNP" (at 214.63 95.25 90)
       (effects (font (size 1.27 1.27)) (justify left))
     )
